File: badge.brd (EAGLE design)
At the start: 77.4 x 72.6 mm, 26 parts, among them U1 TINY2313-*S*, X1 FH12-10S-0.5SH

Commit message: Layout
Parts:
- added R8: (no value), resistor:R0805
- added SJ1: (no value), jumper:SJ
- moved LED6 10.5 mm to (44.0, 80.2)
- moved LED4 0.20 mm to (39.8, 55.9)
Connections:
- new net N$24: R8.1, SJ1.1
- net GND: now also LED4.C
- net N$3: now also SJ1.2
- net N$5: now also R8.2; no longer LED4.C
Routing:
- net N$3: track 44.7 -> 93.5 mm, vias 2 -> 4
- net GND: track 429.0 -> 443.2 mm, vias 7 -> 8
- net N$5: track 18.2 -> 26.2 mm, vias 0 -> 1
- net N$24: track 0.00 -> 2.39 mm
- added copper zone on layer 16, net GND
- removed copper zone on layer 16, net N$28
Other:
- board size 77.4 x 72.6 mm -> 77.4 x 82.9 mm

Commit message: Layout fix
Parts:
- moved R8 12.4 mm to (56.8, 52.6)
- moved SJ1 2.82 mm to (50.0, 52.2), turned to 270 degrees
- turned LED6 to 0 degrees
Routing:
- net GND: track 443.2 -> 255.3 mm, vias 8 -> 7
- net N$5: track 26.2 -> 50.2 mm
- net N$24: track 2.39 -> 7.59 mm
Other:
- outline, holes or cut-outs redrawn
