File: badge.sch (EAGLE design)
At the start: 26 parts, among them U1 TINY2313-*S*, X1 FH12-10S-0.5SH

Commit message: Layout fix
Parts:
- added R8: (no value), resistor:R-EU_R0805
- added SJ1: (no value), jumper:SJ
Connections:
- new net N$24: R8.1, SJ1.1
- net GND: now also LED4.C
- net N$3: now also SJ1.2
- net N$5: now also R8.2; no longer LED4.C
Other:
- moved on the sheet: LED6
Changed lines of the file:
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@@
 <part name="PAD5" library="wirepad" deviceset="WIREPAD" device="SMD1,27-254"/>
 <part name="PAD6" library="wirepad" deviceset="WIREPAD" device="SMD1,27-254"/>
+<part name="R8" library="resistor" deviceset="R-EU_" device="R0805"/>
+<part name="GND9" library="supply1" deviceset="GND" device=""/>
+<part name="SJ1" library="jumper" deviceset="SJ" device=""/>
 </parts>
 <sheets>
@@
 <instance part="G2" gate="G$1" x="-12.7" y="25.4" rot="R90"/>
 <instance part="LED4" gate="G$1" x="86.36" y="55.88" rot="R90"/>
-<instance part="LED6" gate="G$1" x="99.06" y="55.88" rot="R90"/>
+<instance part="LED6" gate="G$1" x="99.06" y="66.04" rot="R90"/>
 <instance part="LED1" gate="G$1" x="78.74" y="48.26" rot="R90"/>
 <instance part="LED2" gate="G$1" x="78.74" y="40.64" rot="R90"/>
 <instance part="LED3" gate="G$1" x="78.74" y="33.02" rot="R90"/>
-<instance part="GND8" gate="1" x="111.76" y="55.88" rot="R90"/>
+<instance part="GND8" gate="1" x="109.22" y="66.04" rot="R90"/>
 <instance part="GND4" gate="1" x="88.9" y="48.26" rot="R90"/>
 <instance part="GND5" gate="1" x="88.9" y="40.64" rot="R90"/>
@@
 <instance part="PAD5" gate="G$1" x="58.42" y="63.5" rot="R270"/>
 <instance part="PAD6" gate="G$1" x="66.04" y="60.96" rot="R270"/>
+<instance part="R8" gate="G$1" x="91.44" y="66.04"/>
+<instance part="GND9" gate="1" x="96.52" y="55.88" rot="R90"/>
+<instance part="SJ1" gate="1" x="78.74" y="66.04" rot="R180"/>
 </instances>
 <busses>
@@
 </segment>
 <segment>
-<pinref part="GND8" gate="1" pin="GND"/>
-<pinref part="LED6" gate="G$1" pin="C"/>
-<wire x1="109.22" y1="55.88" x2="104.14" y2="55.88" width="0.1524" layer="91"/>
-</segment>
-<segment>
 <pinref part="LED1" gate="G$1" pin="C"/>
 <pinref part="GND4" gate="1" pin="GND"/>
@@
 <wire x1="99.06" y1="27.94" x2="93.98" y2="27.94" width="0.1524" layer="91"/>
 </segment>
+<segment>
+<pinref part="LED6" gate="G$1" pin="C"/>
+<pinref part="GND8" gate="1" pin="GND"/>
+<wire x1="104.14" y1="66.04" x2="106.68" y2="66.04" width="0.1524" layer="91"/>
+</segment>
+<segment>
+<pinref part="LED4" gate="G$1" pin="C"/>
+<pinref part="GND9" gate="1" pin="GND"/>
+<wire x1="91.44" y1="55.88" x2="93.98" y2="55.88" width="0.1524" layer="91"/>
+</segment>
 </net>
 <net name="N$2" class="0">
@@
 <wire x1="66.04" y1="58.42" x2="50.8" y2="58.42" width="0.1524" layer="91"/>
 <pinref part="PAD6" gate="G$1" pin="P"/>
+<wire x1="66.04" y1="58.42" x2="71.12" y2="58.42" width="0.1524" layer="91"/>
+<junction x="66.04" y="58.42"/>
+<pinref part="SJ1" gate="1" pin="2"/>
+<wire x1="71.12" y1="58.42" x2="73.66" y2="58.42" width="0.1524" layer="91"/>
+<wire x1="73.66" y1="58.42" x2="73.66" y2="66.04" width="0.1524" layer="91"/>
 </segment>
 </net>
@@
 <wire x1="53.34" y1="63.5" x2="50.8" y2="63.5" width="0.1524" layer="91"/>
 <pinref part="PAD4" gate="G$1" pin="P"/>
-</segment>
-</net>
-<net name="N$5" class="0">
-<segment>
-<pinref part="LED4" gate="G$1" pin="C"/>
-<wire x1="99.06" y1="55.88" x2="96.52" y2="55.88" width="0.1524" layer="91"/>
-<pinref part="LED6" gate="G$1" pin="A"/>
-<wire x1="96.52" y1="55.88" x2="91.44" y2="55.88" width="0.1524" layer="91"/>
-<junction x="96.52" y="55.88"/>
 </segment>
 </net>
@@
 </segment>
 </net>
+<net name="N$5" class="0">
+<segment>
+<pinref part="LED6" gate="G$1" pin="A"/>
+<pinref part="R8" gate="G$1" pin="2"/>
+</segment>
+</net>
+<net name="N$24" class="0">
+<segment>
+<pinref part="R8" gate="G$1" pin="1"/>
+<pinref part="SJ1" gate="1" pin="1"/>
+<wire x1="83.82" y1="66.04" x2="86.36" y2="66.04" width="0.1524" layer="91"/>
+</segment>
+</net>
