File: badge_mil.brd (EAGLE design)
At the start: 77.2 x 83.1 mm, 28 parts, among them U1 TINY2313-*S*, X1 FH12-10S-0.5SH

Commit message: Added jumper as power switch
Parts:
- added SJ2: (no value), jumper:SJ_2W
Connections:
- new net N$28: G2.-, SJ2.3
- net GND: now also SJ2.2; no longer G2.-
Routing:
- net GND: track 180.2 -> 203.6 mm
- net N$28: track 0.00 -> 11.4 mm
Changed lines of the file:
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@@
 </element>
 <element name="SJ1" library="jumper" package="SJW" value="" x="50.508" y="53.216" rot="MR270"/>
+<element name="SJ2" library="jumper" package="SJ_2W" value="" x="65.278" y="39.624" rot="MR270"/>
 </elements>
 <signals>
@@
 <signal name="GND">
 <contactref element="U1" pad="10"/>
-<contactref element="G2" pad="-"/>
 <contactref element="LED1" pad="C"/>
 <contactref element="LED2" pad="C"/>
@@
 <vertex x="1.27" y="43.434"/>
 </polygon>
+<contactref element="SJ2" pad="2"/>
+<wire x1="65.278" y1="39.624" x2="75.438" y2="39.624" width="0.3048" layer="16"/>
+<wire x1="75.438" y1="39.624" x2="75.438" y2="26.924" width="0.3048" layer="16"/>
+<wire x1="75.438" y1="26.924" x2="75.438" y2="26.416" width="0.3048" layer="16"/>
 </signal>
 <signal name="N$2">
@@
 <wire x1="57.15" y1="52.578" x2="57.308" y2="52.766" width="0.254" layer="16"/>
 </signal>
+<signal name="N$28">
+<contactref element="G2" pad="-"/>
+<contactref element="SJ2" pad="3"/>
+<wire x1="69.313" y1="29.731" x2="65.278" y2="29.731" width="0.3048" layer="16"/>
+<wire x1="65.278" y1="29.731" x2="65.278" y2="37.084" width="0.3048" layer="16"/>
+</signal>
 </signals>

Commit message: LCD contrast poti
Parts:
- removed R2: (no value), resistor:R0805
- added R10: (no value), resistor:RTRIM4G/J
- moved SJ2 6.04 mm to (67.6, 45.2), turned to 0 degrees
Connections:
- removed net N$21: R2.1, X1.3
- new net N$42: R10.2, X1.3
- net GND: now also R10.3, X1.1; no longer X1.2
- net VCC: now also R10.1, X1.2; no longer R2.2, X1.1
Routing:
- net N$21: track 23.6 -> 0.00 mm, vias 2 -> 0
- net N$42: track 0.00 -> 22.3 mm, vias 0 -> 2
- net N$28: track 11.4 -> 19.5 mm
- net GND: track 203.6 -> 206.9 mm
- net VCC: track 97.3 -> 96.3 mm
Changed lines of the file:
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@@
 <attribute name="SPICEPREFIX" value="R" x="41.783" y="25.781" size="1.778" layer="28" rot="MR0" display="off"/>
-</element>
-<element name="R2" library="resistor" package="R0805" value="" x="6.223" y="21.971" rot="MR0">
-<attribute name="SPICEPREFIX" value="R" x="6.223" y="21.971" size="1.778" layer="28" rot="MR0" display="off"/>
 </element>
 <element name="R3" library="resistor" package="R0805" value="" x="12.446" y="35.814" rot="MR90">
@@
 </element>
 <element name="SJ1" library="jumper" package="SJW" value="" x="50.508" y="53.216" rot="MR270"/>
-<element name="SJ2" library="jumper" package="SJ_2W" value="" x="65.278" y="39.624" rot="MR270"/>
+<element name="SJ2" library="jumper" package="SJ_2W" value="" x="67.564" y="45.212" rot="MR0"/>
+<element name="R10" library="resistor" package="RTRIM4G/J" value="" x="6.604" y="21.59" rot="MR180"/>
 </elements>
 <signals>
@@
 <contactref element="U1" pad="20"/>
 <contactref element="C1" pad="2"/>
-<contactref element="X1" pad="1"/>
-<contactref element="R2" pad="2"/>
 <wire x1="54.203" y1="6.096" x2="48.3235" y2="6.096" width="0.254" layer="16"/>
 <wire x1="30.008" y1="4.591" x2="29.108" y2="4.591" width="0.254" layer="16"/>
 <wire x1="21.054" y1="12.645" x2="21.054" y2="13.945" width="0.254" layer="16"/>
 <wire x1="21.054" y1="13.945" x2="20.574" y2="14.478" width="0.254" layer="16"/>
-<wire x1="16.764" y1="15.494" x2="19.848" y2="15.494" width="0.254" layer="16"/>
-<wire x1="19.848" y1="15.494" x2="19.848" y2="16.816" width="0.254" layer="16"/>
-<wire x1="5.334" y1="22.098" x2="5.334" y2="23.622" width="0.254" layer="16"/>
-<wire x1="5.334" y1="23.622" x2="8.636" y2="23.622" width="0.254" layer="16"/>
-<wire x1="8.636" y1="23.622" x2="16.764" y2="15.494" width="0.254" layer="16"/>
+<wire x1="16.764" y1="15.494" x2="19.812" y2="15.494" width="0.254" layer="16"/>
+<wire x1="19.812" y1="15.494" x2="19.848" y2="15.494" width="0.254" layer="16"/>
+<wire x1="5.334" y1="22.098" x2="5.588" y2="22.098" width="0.254" layer="16"/>
+<wire x1="5.588" y1="22.098" x2="8.89" y2="22.098" width="0.254" layer="16"/>
+<wire x1="8.89" y1="22.098" x2="16.764" y2="15.494" width="0.254" layer="16"/>
 <contactref element="D1" pad="C"/>
 <wire x1="29.108" y1="4.591" x2="21.054" y2="12.645" width="0.254" layer="16"/>
@@
 <wire x1="3.048" y1="3.556" x2="3.048" y2="22.098" width="0.254" layer="16"/>
 <wire x1="3.048" y1="22.098" x2="5.334" y2="22.098" width="0.254" layer="16"/>
-<wire x1="5.334" y1="22.098" x2="5.373" y2="21.971" width="0.254" layer="16"/>
 <wire x1="29.698" y1="2.966" x2="30.008" y2="2.966" width="0.254" layer="16"/>
 <wire x1="30.008" y1="2.966" x2="30.008" y2="4.591" width="0.254" layer="16"/>
@@
 <wire x1="34.036" y1="3.556" x2="34.008" y2="4.591" width="0.254" layer="16"/>
 <wire x1="20.574" y1="14.478" x2="19.848" y2="15.204" width="0.254" layer="16"/>
-<wire x1="19.848" y1="15.204" x2="19.848" y2="16.816" width="0.254" layer="16"/>
+<contactref element="X1" pad="2"/>
+<wire x1="19.848" y1="15.204" x2="19.812" y2="15.204" width="0.254" layer="16"/>
+<wire x1="19.812" y1="15.204" x2="19.812" y2="15.494" width="0.254" layer="16"/>
+<wire x1="19.812" y1="15.494" x2="20.348" y2="15.494" width="0.254" layer="16"/>
+<wire x1="20.348" y1="15.494" x2="20.348" y2="16.816" width="0.254" layer="16"/>
+<contactref element="R10" pad="1"/>
+<wire x1="5.454" y1="24.34" x2="5.454" y2="22.218" width="0.254" layer="16"/>
+<wire x1="5.454" y1="22.218" x2="5.334" y2="22.098" width="0.254" layer="16"/>
 </signal>
 <signal name="GND">
@@
 <contactref element="LED3" pad="C"/>
 <contactref element="C1" pad="1"/>
-<contactref element="X1" pad="2"/>
 <contactref element="LED5" pad="C"/>
 <wire x1="62.738" y1="55.106" x2="62.738" y2="58.166" width="1.016" layer="1"/>
@@
 </polygon>
 <contactref element="SJ2" pad="2"/>
-<wire x1="65.278" y1="39.624" x2="75.438" y2="39.624" width="0.3048" layer="16"/>
+<wire x1="67.564" y1="45.212" x2="67.564" y2="41.91" width="0.3048" layer="16"/>
+<wire x1="67.564" y1="41.91" x2="67.564" y2="39.624" width="0.3048" layer="16"/>
+<wire x1="67.564" y1="39.624" x2="75.438" y2="39.624" width="0.3048" layer="16"/>
 <wire x1="75.438" y1="39.624" x2="75.438" y2="26.924" width="0.3048" layer="16"/>
 <wire x1="75.438" y1="26.924" x2="75.438" y2="26.416" width="0.3048" layer="16"/>
+<contactref element="X1" pad="1"/>
+<contactref element="R10" pad="3"/>
 </signal>
 <signal name="N$2">
@@
 <wire x1="33.528" y1="21.844" x2="36.576" y2="18.796" width="0.254" layer="16"/>
 </signal>
-<signal name="N$21">
-<contactref element="R2" pad="1"/>
-<contactref element="X1" pad="3"/>
-<wire x1="20.848" y1="16.816" x2="20.848" y2="15.728" width="0.254" layer="16"/>
-<wire x1="20.848" y1="15.728" x2="22.098" y2="14.478" width="0.254" layer="16"/>
-<wire x1="22.098" y1="14.478" x2="22.098" y2="13.208" width="0.254" layer="16"/>
-<via x="22.098" y="13.208" extent="1-16" drill="0.6"/>
-<wire x1="22.098" y1="13.208" x2="19.05" y2="13.208" width="0.254" layer="1"/>
-<via x="19.05" y="13.208" extent="1-16" drill="0.6"/>
-<wire x1="19.05" y1="13.208" x2="14.478" y2="13.208" width="0.254" layer="16"/>
-<wire x1="14.478" y1="13.208" x2="7.112" y2="20.574" width="0.254" layer="16"/>
-<wire x1="7.112" y1="20.574" x2="7.112" y2="21.971" width="0.254" layer="16"/>
-<wire x1="7.112" y1="21.971" x2="7.073" y2="21.971" width="0.254" layer="16"/>
-</signal>
 <signal name="N$22">
 </signal>
@@
 <contactref element="SJ2" pad="3"/>
 <wire x1="69.313" y1="29.731" x2="65.278" y2="29.731" width="0.3048" layer="16"/>
-<wire x1="65.278" y1="29.731" x2="65.278" y2="37.084" width="0.3048" layer="16"/>
+<wire x1="65.278" y1="29.731" x2="65.024" y2="45.212" width="0.3048" layer="16"/>
+</signal>
+<signal name="N$42">
+<contactref element="X1" pad="3"/>
+<wire x1="11.684" y1="14.478" x2="18.542" y2="14.478" width="0.254" layer="16"/>
+<wire x1="18.542" y1="14.478" x2="18.542" y2="13.716" width="0.254" layer="16"/>
+<via x="18.542" y="13.716" extent="1-16" drill="0.6"/>
+<wire x1="18.542" y1="13.716" x2="20.32" y2="13.716" width="0.254" layer="1"/>
+<wire x1="20.32" y1="13.716" x2="21.59" y2="14.986" width="0.254" layer="1"/>
+<via x="21.59" y="14.986" extent="1-16" drill="0.6"/>
+<wire x1="21.59" y1="14.986" x2="21.082" y2="15.494" width="0.254" layer="16"/>
+<wire x1="21.082" y1="15.494" x2="20.828" y2="15.494" width="0.254" layer="16"/>
+<wire x1="20.828" y1="15.494" x2="20.828" y2="16.796" width="0.254" layer="16"/>
+<wire x1="20.828" y1="16.796" x2="20.848" y2="16.816" width="0.254" layer="16"/>
+<contactref element="R10" pad="2"/>
+<wire x1="6.604" y1="18.84" x2="10.624" y2="18.84" width="0.254" layer="16"/>
+<wire x1="10.624" y1="18.84" x2="11.684" y2="17.78" width="0.254" layer="16"/>
+<wire x1="11.684" y1="14.478" x2="11.684" y2="17.78" width="0.254" layer="16"/>
 </signal>
 </signals>

Commit message: Minor changes
Parts:
- D1: value (none) -> LL 5819
- LED1: value Gelb -> Rot
- LED3: value Grün -> Rot
- LED4: value Rot -> Gelb
- LED5: value Rot -> Grün
- R2: value (none) -> 10k
- R3, R4, R5, R6, R7, R8: value (none) -> 1k6
- SJ1: device jumper:SJW -> jumper:SJ_2W
- SJ2: device jumper:SJ_2W -> jumper:SJW
- moved R5 45.0 mm to (64.0, 21.3), turned to 270 degrees
- moved R7 45.0 mm to (31.0, 51.8), turned to 90 degrees
- moved LED3 35.6 mm to (62.7, 54.4), turned to 270 degrees
- moved LED5 35.6 mm to (27.2, 52.5), turned to 90 degrees
- moved LED1 34.1 mm to (40.1, 56.9)
- moved R3 31.0 mm to (41.8, 25.8), turned to 0 degrees
- moved R6 31.0 mm to (14.5, 40.4), turned to 90 degrees
- moved LED4 22.5 mm to (17.7, 58.2)
- moved SJ1 18.8 mm to (67.6, 45.2), turned to 0 degrees
- moved SJ2 18.8 mm to (50.5, 53.2), turned to 270 degrees
- moved LED2 12.5 mm to (6.22, 53.1)
- moved R4 5.00 mm to (12.4, 35.8)
- renumbered R10 to R2
Connections:
- net GND: now also SJ1.2; no longer SJ2.2
- net N$10: now also R3.1; no longer R6.1
- net N$11: now also R4.1; no longer R3.1
- net N$12: now also R6.1; no longer R4.1
- net N$13: now also R7.1; no longer R5.1
- net N$24: now also SJ2.1; no longer SJ1.1
- net N$28: now also SJ1.3; no longer SJ2.3
- net N$3: now also SJ2.2; no longer SJ1.2
- net N$39: now also LED3.A, R5.1; no longer LED5.A, R7.1
- net N$40: now also R5.2; no longer R7.2
- net N$6: now also LED5.A, R7.2; no longer LED3.A, R5.2
Routing:
- net N$36: track 18.6 -> 57.8 mm, vias 1 -> 2
- net N$7: track 56.7 -> 18.6 mm, vias 2 -> 1
- net N$9: track 57.8 -> 56.7 mm
