File: badge_mil.sch (EAGLE design)
At the start: 28 parts, among them U1 TINY2313-*S*, X1 FH12-10S-0.5SH

Commit message: Resistor Package
Parts:
- R3: device resistor:R-EU_R0603 -> resistor:R-EU_R0805
- SJ1: device jumper:SJ -> jumper:SJW
Changed lines of the file:
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@@
 <?xml version="1.0" encoding="utf-8"?>
 <!DOCTYPE eagle SYSTEM "eagle.dtd">
-<eagle version="7.2.0">
+<eagle version="7.1.0">
 <drawing>
 <settings>
@@
 <grid distance="0.1" unitdist="inch" unit="inch" style="lines" multiple="1" display="no" altdistance="0.01" altunitdist="inch" altunit="inch"/>
 <layers>
-<layer number="1" name="Top" color="4" fill="1" visible="no" active="no"/>
-<layer number="16" name="Bottom" color="1" fill="1" visible="no" active="no"/>
-<layer number="17" name="Pads" color="2" fill="1" visible="no" active="no"/>
-<layer number="18" name="Vias" color="2" fill="1" visible="no" active="no"/>
-<layer number="19" name="Unrouted" color="6" fill="1" visible="no" active="no"/>
-<layer number="20" name="Dimension" color="15" fill="1" visible="no" active="no"/>
-<layer number="21" name="tPlace" color="7" fill="1" visible="no" active="no"/>
-<layer number="22" name="bPlace" color="7" fill="1" visible="no" active="no"/>
-<layer number="23" name="tOrigins" color="15" fill="1" visible="no" active="no"/>
-<layer number="24" name="bOrigins" color="15" fill="1" visible="no" active="no"/>
-<layer number="25" name="tNames" color="7" fill="1" visible="no" active="no"/>
-<layer number="26" name="bNames" color="7" fill="1" visible="no" active="no"/>
-<layer number="27" name="tValues" color="7" fill="1" visible="no" active="no"/>
-<layer number="28" name="bValues" color="7" fill="1" visible="no" active="no"/>
+<layer number="1" name="Top" color="4" fill="1" visible="yes" active="no"/>
+<layer number="16" name="Bottom" color="1" fill="1" visible="yes" active="no"/>
+<layer number="17" name="Pads" color="2" fill="1" visible="yes" active="no"/>
+<layer number="18" name="Vias" color="2" fill="1" visible="yes" active="no"/>
+<layer number="19" name="Unrouted" color="6" fill="1" visible="yes" active="no"/>
+<layer number="20" name="Dimension" color="15" fill="1" visible="yes" active="no"/>
+<layer number="21" name="tPlace" color="7" fill="1" visible="yes" active="no"/>
+<layer number="22" name="bPlace" color="7" fill="1" visible="yes" active="no"/>
+<layer number="23" name="tOrigins" color="15" fill="1" visible="yes" active="no"/>
+<layer number="24" name="bOrigins" color="15" fill="1" visible="yes" active="no"/>
+<layer number="25" name="tNames" color="7" fill="1" visible="yes" active="no"/>
+<layer number="26" name="bNames" color="7" fill="1" visible="yes" active="no"/>
+<layer number="27" name="tValues" color="7" fill="1" visible="yes" active="no"/>
+<layer number="28" name="bValues" color="7" fill="1" visible="yes" active="no"/>
 <layer number="29" name="tStop" color="7" fill="3" visible="no" active="no"/>
 <layer number="30" name="bStop" color="7" fill="6" visible="no" active="no"/>
@@
 <layer number="35" name="tGlue" color="7" fill="4" visible="no" active="no"/>
 <layer number="36" name="bGlue" color="7" fill="5" visible="no" active="no"/>
-<layer number="37" name="tTest" color="7" fill="1" visible="no" active="no"/>
-<layer number="38" name="bTest" color="7" fill="1" visible="no" active="no"/>
+<layer number="37" name="tTest" color="7" fill="1" visible="yes" active="no"/>
+<layer number="38" name="bTest" color="7" fill="1" visible="yes" active="no"/>
 <layer number="39" name="tKeepout" color="4" fill="11" visible="no" active="no"/>
 <layer number="40" name="bKeepout" color="1" fill="11" visible="no" active="no"/>
@@
 <layer number="44" name="Drills" color="7" fill="1" visible="no" active="no"/>
 <layer number="45" name="Holes" color="7" fill="1" visible="no" active="no"/>
-<layer number="46" name="Milling" color="3" fill="1" visible="no" active="no"/>
-<layer number="47" name="Measures" color="7" fill="1" visible="no" active="no"/>
-<layer number="48" name="Document" color="7" fill="1" visible="no" active="no"/>
-<layer number="49" name="Reference" color="7" fill="1" visible="no" active="no"/>
-<layer number="50" name="dxf" color="7" fill="1" visible="no" active="no"/>
-<layer number="51" name="tDocu" color="7" fill="1" visible="no" active="no"/>
-<layer number="52" name="bDocu" color="7" fill="1" visible="no" active="no"/>
+<layer number="46" name="Milling" color="3" fill="1" visible="yes" active="no"/>
+<layer number="47" name="Measures" color="7" fill="1" visible="yes" active="no"/>
+<layer number="48" name="Document" color="7" fill="1" visible="yes" active="no"/>
+<layer number="49" name="Reference" color="7" fill="1" visible="yes" active="no"/>
+<layer number="50" name="dxf" color="7" fill="1" visible="yes" active="no"/>
+<layer number="51" name="tDocu" color="7" fill="1" visible="yes" active="no"/>
+<layer number="52" name="bDocu" color="7" fill="1" visible="yes" active="no"/>
 <layer number="90" name="Modules" color="5" fill="1" visible="yes" active="yes"/>
 <layer number="91" name="Nets" color="2" fill="1" visible="yes" active="yes"/>
@@
 <part name="R6" library="resistor" deviceset="R-EU_" device="R0805"/>
 <part name="R2" library="resistor" deviceset="R-EU_" device="R0805"/>
-<part name="R3" library="resistor" deviceset="R-EU_" device="R0603"/>
+<part name="R3" library="resistor" deviceset="R-EU_" device="R0805"/>
 <part name="R4" library="resistor" deviceset="R-EU_" device="R0805"/>
 <part name="R5" library="resistor" deviceset="R-EU_" device="R0805"/>
@@
 <part name="R8" library="resistor" deviceset="R-EU_" device="R0805"/>
 <part name="GND9" library="supply1" deviceset="GND" device=""/>
-<part name="SJ1" library="jumper" deviceset="SJ" device=""/>
+<part name="SJ1" library="jumper" deviceset="SJ" device="W"/>
 </parts>
 <sheets>

Commit message: Added jumper as power switch
Parts:
- added SJ2: (no value), jumper:SJ2WW
Connections:
- new net N$28: G2.-, SJ2.3
- net GND: now also SJ2.2; no longer G2.-
Changed lines of the file:
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@@
 <grid distance="0.1" unitdist="inch" unit="inch" style="lines" multiple="1" display="no" altdistance="0.01" altunitdist="inch" altunit="inch"/>
 <layers>
-<layer number="1" name="Top" color="4" fill="1" visible="yes" active="no"/>
-<layer number="16" name="Bottom" color="1" fill="1" visible="yes" active="no"/>
-<layer number="17" name="Pads" color="2" fill="1" visible="yes" active="no"/>
-<layer number="18" name="Vias" color="2" fill="1" visible="yes" active="no"/>
-<layer number="19" name="Unrouted" color="6" fill="1" visible="yes" active="no"/>
-<layer number="20" name="Dimension" color="15" fill="1" visible="yes" active="no"/>
-<layer number="21" name="tPlace" color="7" fill="1" visible="yes" active="no"/>
-<layer number="22" name="bPlace" color="7" fill="1" visible="yes" active="no"/>
-<layer number="23" name="tOrigins" color="15" fill="1" visible="yes" active="no"/>
-<layer number="24" name="bOrigins" color="15" fill="1" visible="yes" active="no"/>
-<layer number="25" name="tNames" color="7" fill="1" visible="yes" active="no"/>
-<layer number="26" name="bNames" color="7" fill="1" visible="yes" active="no"/>
-<layer number="27" name="tValues" color="7" fill="1" visible="yes" active="no"/>
-<layer number="28" name="bValues" color="7" fill="1" visible="yes" active="no"/>
+<layer number="1" name="Top" color="4" fill="1" visible="no" active="no"/>
+<layer number="16" name="Bottom" color="1" fill="1" visible="no" active="no"/>
+<layer number="17" name="Pads" color="2" fill="1" visible="no" active="no"/>
+<layer number="18" name="Vias" color="2" fill="1" visible="no" active="no"/>
+<layer number="19" name="Unrouted" color="6" fill="1" visible="no" active="no"/>
+<layer number="20" name="Dimension" color="15" fill="1" visible="no" active="no"/>
+<layer number="21" name="tPlace" color="7" fill="1" visible="no" active="no"/>
+<layer number="22" name="bPlace" color="7" fill="1" visible="no" active="no"/>
+<layer number="23" name="tOrigins" color="15" fill="1" visible="no" active="no"/>
+<layer number="24" name="bOrigins" color="15" fill="1" visible="no" active="no"/>
+<layer number="25" name="tNames" color="7" fill="1" visible="no" active="no"/>
+<layer number="26" name="bNames" color="7" fill="1" visible="no" active="no"/>
+<layer number="27" name="tValues" color="7" fill="1" visible="no" active="no"/>
+<layer number="28" name="bValues" color="7" fill="1" visible="no" active="no"/>
 <layer number="29" name="tStop" color="7" fill="3" visible="no" active="no"/>
 <layer number="30" name="bStop" color="7" fill="6" visible="no" active="no"/>
@@
 <layer number="35" name="tGlue" color="7" fill="4" visible="no" active="no"/>
 <layer number="36" name="bGlue" color="7" fill="5" visible="no" active="no"/>
-<layer number="37" name="tTest" color="7" fill="1" visible="yes" active="no"/>
-<layer number="38" name="bTest" color="7" fill="1" visible="yes" active="no"/>
+<layer number="37" name="tTest" color="7" fill="1" visible="no" active="no"/>
+<layer number="38" name="bTest" color="7" fill="1" visible="no" active="no"/>
 <layer number="39" name="tKeepout" color="4" fill="11" visible="no" active="no"/>
 <layer number="40" name="bKeepout" color="1" fill="11" visible="no" active="no"/>
@@
 <layer number="44" name="Drills" color="7" fill="1" visible="no" active="no"/>
 <layer number="45" name="Holes" color="7" fill="1" visible="no" active="no"/>
-<layer number="46" name="Milling" color="3" fill="1" visible="yes" active="no"/>
-<layer number="47" name="Measures" color="7" fill="1" visible="yes" active="no"/>
-<layer number="48" name="Document" color="7" fill="1" visible="yes" active="no"/>
-<layer number="49" name="Reference" color="7" fill="1" visible="yes" active="no"/>
-<layer number="50" name="dxf" color="7" fill="1" visible="yes" active="no"/>
-<layer number="51" name="tDocu" color="7" fill="1" visible="yes" active="no"/>
-<layer number="52" name="bDocu" color="7" fill="1" visible="yes" active="no"/>
+<layer number="46" name="Milling" color="3" fill="1" visible="no" active="no"/>
+<layer number="47" name="Measures" color="7" fill="1" visible="no" active="no"/>
+<layer number="48" name="Document" color="7" fill="1" visible="no" active="no"/>
+<layer number="49" name="Reference" color="7" fill="1" visible="no" active="no"/>
+<layer number="50" name="dxf" color="7" fill="1" visible="no" active="no"/>
+<layer number="51" name="tDocu" color="7" fill="1" visible="no" active="no"/>
+<layer number="52" name="bDocu" color="7" fill="1" visible="no" active="no"/>
 <layer number="90" name="Modules" color="5" fill="1" visible="yes" active="yes"/>
 <layer number="91" name="Nets" color="2" fill="1" visible="yes" active="yes"/>
@@
 <part name="GND9" library="supply1" deviceset="GND" device=""/>
 <part name="SJ1" library="jumper" deviceset="SJ" device="W"/>
+<part name="SJ2" library="jumper" deviceset="SJ2W" device="W"/>
 </parts>
 <sheets>
@@
 <instance part="GND9" gate="1" x="96.52" y="55.88" rot="R90"/>
 <instance part="SJ1" gate="1" x="78.74" y="66.04" rot="R180"/>
+<instance part="SJ2" gate="G$1" x="-12.7" y="10.16" rot="R180"/>
 </instances>
 <busses>
@@
 <wire x1="7.62" y1="20.32" x2="7.62" y2="17.78" width="0.1524" layer="91"/>
 <junction x="7.62" y="20.32"/>
-<pinref part="G2" gate="G$1" pin="-"/>
-<wire x1="7.62" y1="17.78" x2="-12.7" y2="17.78" width="0.1524" layer="91"/>
-<wire x1="-12.7" y1="17.78" x2="-12.7" y2="20.32" width="0.1524" layer="91"/>
 <pinref part="PAD2" gate="G$1" pin="P"/>
+<pinref part="SJ2" gate="G$1" pin="2"/>
+<wire x1="-7.62" y1="10.16" x2="7.62" y2="10.16" width="0.1524" layer="91"/>
+<wire x1="7.62" y1="10.16" x2="7.62" y2="17.78" width="0.1524" layer="91"/>
 </segment>
 <segment>
@@
 </segment>
 </net>
+<net name="N$28" class="0">
+<segment>
+<pinref part="G2" gate="G$1" pin="-"/>
+<wire x1="-12.7" y1="17.78" x2="-12.7" y2="20.32" width="0.1524" layer="91"/>
+<pinref part="SJ2" gate="G$1" pin="3"/>
+<wire x1="-12.7" y1="15.24" x2="-12.7" y2="17.78" width="0.1524" layer="91"/>
+</segment>
+</net>

Commit message: LCD contrast poti
Parts:
- removed R2: (no value), resistor:R-EU_R0805
- added R10: (no value), resistor:R-TRIMM4G/J
Connections:
- removed net N$21: R2.1, X1-3.1
- new net N$42: R10.S, X1-3.1
- net GND: now also R10.A, X1-1.1; no longer X1-2.1
- net VCC: now also R10.E, X1-2.1; no longer R2.2, X1-1.1
Other:
- moved on the sheet: LED2, LED4, LED5, R4, R6, R7, X1-3
Changed lines of the file:
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@@
 <setting verticaltext="up"/>
 </settings>
-<grid distance="0.1" unitdist="inch" unit="inch" style="lines" multiple="1" display="no" altdistance="0.01" altunitdist="inch" altunit="inch"/>
+<grid distance="10" unitdist="mil" unit="mil" style="lines" multiple="1" display="yes" altdistance="0.01" altunitdist="inch" altunit="inch"/>
 <layers>
 <layer number="1" name="Top" color="4" fill="1" visible="no" active="no"/>
@@
 <part name="GND1" library="supply1" deviceset="GND" device=""/>
 <part name="R6" library="resistor" deviceset="R-EU_" device="R0805"/>
-<part name="R2" library="resistor" deviceset="R-EU_" device="R0805"/>
 <part name="R3" library="resistor" deviceset="R-EU_" device="R0805"/>
 <part name="R4" library="resistor" deviceset="R-EU_" device="R0805"/>
@@
 <part name="SJ1" library="jumper" deviceset="SJ" device="W"/>
 <part name="SJ2" library="jumper" deviceset="SJ2W" device="W"/>
+<part name="R10" library="resistor" deviceset="R-TRIMM" device="4G/J"/>
+<part name="GND10" library="supply1" deviceset="GND" device=""/>
 </parts>
 <sheets>
@@
 <instance part="GND2" gate="1" x="12.7" y="17.78"/>
 <instance part="G2" gate="G$1" x="-12.7" y="25.4" rot="R90"/>
-<instance part="LED4" gate="G$1" x="86.36" y="55.88" rot="R90"/>
+<instance part="LED4" gate="G$1" x="78.74" y="55.626" rot="R90"/>
 <instance part="LED6" gate="G$1" x="99.06" y="66.04" rot="R90"/>
 <instance part="LED1" gate="G$1" x="78.74" y="48.26" rot="R90"/>
-<instance part="LED2" gate="G$1" x="78.74" y="40.64" rot="R90"/>
+<instance part="LED2" gate="G$1" x="78.74" y="37.846" rot="R90"/>
 <instance part="LED3" gate="G$1" x="78.74" y="33.02" rot="R90"/>
 <instance part="GND8" gate="1" x="109.22" y="66.04" rot="R90"/>
 <instance part="GND4" gate="1" x="88.9" y="48.26" rot="R90"/>
-<instance part="GND5" gate="1" x="88.9" y="40.64" rot="R90"/>
+<instance part="GND5" gate="1" x="88.9" y="37.846" rot="R90"/>
 <instance part="GND6" gate="1" x="88.9" y="33.02" rot="R90"/>
 <instance part="C1" gate="G$1" x="-10.16" y="60.96" rot="R180"/>
 <instance part="GND1" gate="1" x="-10.16" y="53.34"/>
-<instance part="R6" gate="G$1" x="71.12" y="55.88"/>
-<instance part="R2" gate="G$1" x="40.64" y="7.62" rot="R90"/>
+<instance part="R6" gate="G$1" x="65.786" y="55.626"/>
 <instance part="R3" gate="G$1" x="66.04" y="48.26"/>
-<instance part="R4" gate="G$1" x="66.04" y="40.64"/>
-<instance part="R5" gate="G$1" x="66.04" y="33.02"/>
+<instance part="R4" gate="G$1" x="66.04" y="37.846"/>
+<instance part="R5" gate="G$1" x="66.294" y="33.02"/>
 <instance part="X1" gate="-1" x="55.88" y="2.54" rot="R90"/>
 <instance part="X1" gate="-2" x="63.5" y="2.54" rot="R90"/>
-<instance part="X1" gate="-3" x="40.64" y="-5.08" rot="R270"/>
+<instance part="X1" gate="-3" x="40.64" y="-15.24" rot="R270"/>
 <instance part="X1" gate="-4" x="50.8" y="40.64" rot="R90"/>
 <instance part="X1" gate="-5" x="53.34" y="40.64" rot="R90"/>
@@
 <instance part="X1" gate="-9" x="58.42" y="25.4" rot="MR180"/>
 <instance part="X1" gate="-10" x="58.42" y="27.94" rot="MR180"/>
-<instance part="GND3" gate="1" x="63.5" y="-5.08"/>
-<instance part="P+3" gate="VCC" x="55.88" y="-5.08" rot="R180"/>
+<instance part="GND3" gate="1" x="55.88" y="-5.08"/>
+<instance part="P+3" gate="VCC" x="63.5" y="-5.08" rot="R180"/>
 <instance part="P+2" gate="VCC" x="48.26" y="15.24" rot="R270"/>
-<instance part="LED5" gate="G$1" x="88.9" y="27.94" rot="R90"/>
-<instance part="GND7" gate="1" x="101.6" y="27.94" rot="R90"/>
-<instance part="R7" gate="G$1" x="76.2" y="27.94" rot="R180"/>
+<instance part="LED5" gate="G$1" x="78.74" y="43.18" rot="R90"/>
+<instance part="GND7" gate="1" x="88.9" y="43.18" rot="R90"/>
+<instance part="R7" gate="G$1" x="66.04" y="43.18" rot="R180"/>
 <instance part="G1" gate="G$1" x="-12.7" y="38.1" rot="R90"/>
 <instance part="D1" gate="G$1" x="-12.7" y="48.26" rot="R90"/>
@@
 <instance part="PAD6" gate="G$1" x="66.04" y="60.96" rot="R270"/>
 <instance part="R8" gate="G$1" x="91.44" y="66.04"/>
-<instance part="GND9" gate="1" x="96.52" y="55.88" rot="R90"/>
+<instance part="GND9" gate="1" x="88.9" y="55.626" rot="R90"/>
 <instance part="SJ1" gate="1" x="78.74" y="66.04" rot="R180"/>
 <instance part="SJ2" gate="G$1" x="-12.7" y="10.16" rot="R180"/>
+<instance part="R10" gate="G$1" x="40.64" y="7.62" rot="R180"/>
+<instance part="GND10" gate="1" x="40.64" y="0"/>
 </instances>
 <busses>
@@
 </segment>
 <segment>
-<pinref part="P+3" gate="VCC" pin="VCC"/>
-<pinref part="X1" gate="-1" pin="1"/>
-<wire x1="55.88" y1="-2.54" x2="55.88" y2="0" width="0.1524" layer="91"/>
-</segment>
-<segment>
 <pinref part="P+2" gate="VCC" pin="VCC"/>
-<pinref part="R2" gate="G$1" pin="2"/>
 <wire x1="45.72" y1="15.24" x2="40.64" y2="15.24" width="0.1524" layer="91"/>
 <wire x1="40.64" y1="15.24" x2="40.64" y2="12.7" width="0.1524" layer="91"/>
+<pinref part="R10" gate="G$1" pin="E"/>
+</segment>
+<segment>
+<pinref part="P+3" gate="VCC" pin="VCC"/>
+<pinref part="X1" gate="-2" pin="1"/>
+<wire x1="63.5" y1="-2.54" x2="63.5" y2="0" width="0.1524" layer="91"/>
 </segment>
 </net>
@@
 <pinref part="LED2" gate="G$1" pin="C"/>
 <pinref part="GND5" gate="1" pin="GND"/>
-<wire x1="83.82" y1="40.64" x2="86.36" y2="40.64" width="0.1524" layer="91"/>
+<wire x1="83.82" y1="37.846" x2="86.36" y2="37.846" width="0.1524" layer="91"/>
 </segment>
 <segment>
@@
 </segment>
 <segment>
-<pinref part="GND3" gate="1" pin="GND"/>
-<pinref part="X1" gate="-2" pin="1"/>
-<wire x1="63.5" y1="-2.54" x2="63.5" y2="0" width="0.1524" layer="91"/>
-</segment>
-<segment>
 <pinref part="GND7" gate="1" pin="GND"/>
 <pinref part="LED5" gate="G$1" pin="C"/>
-<wire x1="99.06" y1="27.94" x2="93.98" y2="27.94" width="0.1524" layer="91"/>
+<wire x1="86.36" y1="43.18" x2="83.82" y2="43.18" width="0.1524" layer="91"/>
 </segment>
 <segment>
@@
 <pinref part="LED4" gate="G$1" pin="C"/>
 <pinref part="GND9" gate="1" pin="GND"/>
-<wire x1="91.44" y1="55.88" x2="93.98" y2="55.88" width="0.1524" layer="91"/>
+<wire x1="83.82" y1="55.626" x2="86.36" y2="55.626" width="0.1524" layer="91"/>
+</segment>
+<segment>
+<pinref part="GND3" gate="1" pin="GND"/>
+<pinref part="X1" gate="-1" pin="1"/>
+<wire x1="55.88" y1="-2.54" x2="55.88" y2="0" width="0.1524" layer="91"/>
+</segment>
+<segment>
+<pinref part="R10" gate="G$1" pin="A"/>
+<pinref part="GND10" gate="1" pin="GND"/>
 </segment>
 </net>
@@
 <pinref part="LED3" gate="G$1" pin="A"/>
 <pinref part="R5" gate="G$1" pin="2"/>
-<wire x1="76.2" y1="33.02" x2="71.12" y2="33.02" width="0.1524" layer="91"/>
+<wire x1="76.2" y1="33.02" x2="71.374" y2="33.02" width="0.1524" layer="91"/>
 </segment>
 </net>
@@
 <pinref part="LED2" gate="G$1" pin="A"/>
 <pinref part="R4" gate="G$1" pin="2"/>
-<wire x1="76.2" y1="40.64" x2="71.12" y2="40.64" width="0.1524" layer="91"/>
+<wire x1="76.2" y1="37.846" x2="71.12" y2="37.846" width="0.1524" layer="91"/>
 </segment>
 </net>
@@
 <pinref part="R6" gate="G$1" pin="2"/>
 <pinref part="LED4" gate="G$1" pin="A"/>
-<wire x1="76.2" y1="55.88" x2="83.82" y2="55.88" width="0.1524" layer="91"/>
+<wire x1="70.866" y1="55.626" x2="76.2" y2="55.626" width="0.1524" layer="91"/>
 </segment>
 </net>
@@
 <pinref part="R6" gate="G$1" pin="1"/>
 <pinref part="U1" gate="G$1" pin="(OC1B)PB4"/>
-<wire x1="66.04" y1="55.88" x2="50.8" y2="55.88" width="0.1524" layer="91"/>
+<wire x1="60.706" y1="55.626" x2="50.8" y2="55.88" width="0.1524" layer="91"/>
 </segment>
 </net>
@@
 <segment>
 <pinref part="R4" gate="G$1" pin="1"/>
-<wire x1="60.96" y1="40.64" x2="58.42" y2="40.64" width="0.1524" layer="91"/>
-<wire x1="58.42" y1="40.64" x2="58.42" y2="50.8" width="0.1524" layer="91"/>
+<wire x1="60.96" y1="37.846" x2="58.42" y2="37.846" width="0.1524" layer="91"/>
+<wire x1="58.42" y1="37.846" x2="58.42" y2="50.8" width="0.1524" layer="91"/>
 <pinref part="U1" gate="G$1" pin="(OC0A)PB2"/>
 <wire x1="58.42" y1="50.8" x2="50.8" y2="50.8" width="0.1524" layer="91"/>
@@
 <segment>
 <pinref part="R5" gate="G$1" pin="1"/>
-<wire x1="60.96" y1="33.02" x2="55.88" y2="33.02" width="0.1524" layer="91"/>
+<wire x1="61.214" y1="33.02" x2="55.88" y2="33.02" width="0.1524" layer="91"/>
 <wire x1="55.88" y1="33.02" x2="55.88" y2="48.26" width="0.1524" layer="91"/>
 <pinref part="U1" gate="G$1" pin="(AIN1)PB1"/>
@@
 </segment>
 </net>
-<net name="N$21" class="0">
-<segment>
-<pinref part="R2" gate="G$1" pin="1"/>
-<pinref part="X1" gate="-3" pin="1"/>
-<wire x1="40.64" y1="-2.54" x2="40.64" y2="2.54" width="0.1524" layer="91"/>
-</segment>
-</net>
 <net name="N$39" class="0">
 <segment>
 <pinref part="LED5" gate="G$1" pin="A"/>
 <pinref part="R7" gate="G$1" pin="1"/>
-<wire x1="86.36" y1="27.94" x2="81.28" y2="27.94" width="0.1524" layer="91"/>
+<wire x1="76.2" y1="43.18" x2="71.12" y2="43.18" width="0.1524" layer="91"/>
 </segment>
 </net>
@@
 <segment>
 <pinref part="R7" gate="G$1" pin="2"/>
-<wire x1="71.12" y1="27.94" x2="71.12" y2="45.72" width="0.1524" layer="91"/>
+<wire x1="60.96" y1="43.18" x2="60.96" y2="45.72" width="0.1524" layer="91"/>
 <pinref part="U1" gate="G$1" pin="(AIN0)PB0"/>
-<wire x1="71.12" y1="45.72" x2="50.8" y2="45.72" width="0.1524" layer="91"/>
+<wire x1="60.96" y1="45.72" x2="50.8" y2="45.72" width="0.1524" layer="91"/>
 </segment>
 </net>
@@
 </segment>
 </net>
+<net name="N$42" class="0">
+<segment>
+<pinref part="X1" gate="-3" pin="1"/>
+<wire x1="40.64" y1="-10.16" x2="40.64" y2="-12.7" width="0.1524" layer="91"/>
+<pinref part="R10" gate="G$1" pin="S"/>
+<wire x1="35.56" y1="7.62" x2="35.56" y2="-10.16" width="0.1524" layer="91"/>
+<wire x1="35.56" y1="-10.16" x2="40.64" y2="-10.16" width="0.1524" layer="91"/>
+</segment>
+</net>

Commit message: Minor changes
Parts:
- D1: value (none) -> LL 5819
- LED1: value Gelb -> Rot
- LED3: value Grün -> Rot
- LED4: value Rot -> Gelb
- LED5: value Rot -> Grün
- R2: value (none) -> 10k
- R3, R4, R5, R6, R7, R8: value (none) -> 1k6
- SJ1: device jumper:SJW -> jumper:SJ2WW
- SJ2: device jumper:SJ2WW -> jumper:SJW
- renumbered R10 to R2
Connections:
- net GND: now also SJ1.2; no longer SJ2.2
- net N$10: now also R3.1; no longer R6.1
- net N$11: now also R4.1; no longer R3.1
- net N$12: now also R6.1; no longer R4.1
- net N$13: now also R7.1; no longer R5.1
- net N$24: now also SJ2.1; no longer SJ1.1
- net N$28: now also SJ1.3; no longer SJ2.3
- net N$3: now also SJ2.2; no longer SJ1.2
- net N$39: now also LED3.A, R5.1; no longer LED5.A, R7.1
- net N$40: now also R5.2; no longer R7.2
- net N$6: now also LED5.A, R7.2; no longer LED3.A, R5.2
Other:
- moved on the sheet: LED1, LED2, LED3, LED4, LED5, R3, R4, R5, R6, R7
