File: eagle/badge_mil.brd (EAGLE design)
At the start: 77.2 x 83.1 mm, 31 parts, among them U1 TINY2313-*S*, X1 FH12-10S-0.5S

Commit message: Minor adjustments for production
Parts:
- U2: value (none) -> MC5205
- renumbered U$1 to CLIP2, U$2 to CLIP1
Other:
- outline, holes or cut-outs redrawn
